Commit message: Updated pick and place movement of arm for experimentation

File: src/mobman_description/control/ros2_control.xacro (robot description, xacro)
@@ -73,6 +73,8 @@
       </joint>
       <joint name="${prefix}gripper_right_joint">
-        <param name="mimic">${prefix}gripper_left_joint</param>
-        <param name="multiplier">1.0</param>
+        <command_interface name="position">
+          <param name="min">-0.010</param>
+          <param name="max">0.019</param>
+        </command_interface>
         <state_interface name="position">
           <param name="initial_value">0.0</param>

File: src/mobman_description/urdf/open_manipulator_x.urdf.xacro (robot description, xacro)
@@ -193,5 +193,4 @@
       <axis xyz="0 -1 0" />
       <limit velocity="4.8" effort="1" lower="-0.010" upper="0.019" />
-      <mimic joint="${prefix}gripper_left_joint" multiplier="1" />
       <dynamics damping="0.1" />
     </joint>

File: src/mobman_description/urdf/turtlebot3_waffle_pi.urdf.xacro (robot description, xacro)
@@ -207,5 +207,5 @@
         <origin xyz="0.015 0 -0.0065" rpy="0 0 0" />
         <geometry>
-          <cylinder length="0.0315" radius="0.055" />
+          <mesh filename="${meshes_file_direction}/ladar.stl" scale="0.001 0.001 0.001" />
         </geometry>
       </collision>
