Commit message: Tryingout few things, may work may not

File: src/mobman_description/urdf/gazebo_plgn.xacro (robot description, xacro)
@@ -40,5 +40,4 @@
       <topic>/cmd_vel</topic>
       <odom_topic>/odom</odom_topic>
-      <tf_topic>/tf</tf_topic>
       <frame_id>odom</frame_id>
       <child_frame_id>base_footprint</child_frame_id>
@@ -125,11 +124,11 @@
     </sensor>
   </gazebo>
-  <gazebo reference="camera_rgb_frame">
-    <sensor name="depth_camera" type="rgbd_camera">
+  <gazebo reference="intel_camera_color_optical_frame">
+    <sensor name="intel_depth_camera" type="rgbd_camera">
       <always_on>true</always_on>
       <visualize>true</visualize>
       <update_rate>5.0</update_rate>
-      <topic>/depth_camera</topic>
-      <gz_frame_id>camera_link</gz_frame_id>
+      <topic>intel_camera</topic>
+      <gz_frame_id>intel_camera_color_optical_frame</gz_frame_id>
       <camera>
         <horizontal_fov>1.047198</horizontal_fov>
@@ -137,23 +136,14 @@
           <width>640</width>
           <height>480</height>
+          <format>R8G8B8</format>
         </image>
         <clip>
           <near>0.05</near>
-          <far>3</far>
+          <far>10.0</far>
         </clip>
+        <depth_camera>
+          <output>depths</output>
+        </depth_camera>
       </camera>
-      <baseline>0.2</baseline>
-      <pointCloudCutoff>0.5</pointCloudCutoff>
-      <pointCloudCutoffMax>3.0</pointCloudCutoffMax>
-      <distortionK1>0</distortionK1>
-      <distortionK2>0</distortionK2>
-      <distortionK3>0</distortionK3>
-      <distortionT1>0</distortionT1>
-      <distortionT2>0</distortionT2>
-      <CxPrime>0</CxPrime>
-      <Cx>0</Cx>
-      <Cy>0</Cy>
-      <focalLength>0</focalLength>
-      <hackBaseline>0</hackBaseline>
     </sensor>
   </gazebo>

File: src/mobman_description/urdf/open_manipulator_x.urdf.xacro (robot description, xacro)
@@ -152,4 +152,41 @@
       </inertial>
     </link>
+    <joint name="${prefix}intel_cam_joint" type="fixed">
+      <parent link="${prefix}link5" />
+      <child link="${prefix}intel_camera" />
+      <origin xyz="0.04 0.0 0.05" rpy="0 0 0" />
+    </joint>
+    <link name="${prefix}intel_camera">
+      <visual>
+        <origin xyz="0 0 0" rpy="${pi/2} 0 ${pi/2}" />
+        <geometry>
+          <mesh filename="${meshes_file_direction}/intelcam/d455.stl" scale="0.001 0.001 0.001"/>
+        </geometry>
+        <material name="grey" />
+      </visual>
+      <collision>
+        <origin xyz="0 0 0" rpy="${pi/2} 0 ${pi/2}" />
+        <geometry>
+          <mesh filename="${meshes_file_direction}/intelcam/d455.stl" scale="0.001 0.001 0.001"/>
+        </geometry>
+      </collision>
+      <inertial>
+        <origin xyz="0 0 0" rpy="0 0 0"/>
+        <mass value="0.072"/>
+        <inertia ixx="1e-4" ixy="0" ixz="0" iyy="1e-4" iyz="0" izz="1e-4"/>
+      </inertial>
+    </link>
+    <joint name="${prefix}intel_camera_color_optical_joint" type="fixed">
+      <parent link="${prefix}intel_camera" />
+      <child link="${prefix}intel_camera_color_optical_frame" />
+      <origin xyz="0 0 0" rpy="0 0 0" />
+    </joint>
+    <link name="${prefix}intel_camera_color_optical_frame" />
+    <joint name="${prefix}intel_camera_depth_optical_joint" type="fixed">
+      <parent link="${prefix}intel_camera_color_optical_frame" />
+      <child link="${prefix}intel_camera_depth_optical_frame" />
+      <origin xyz="0 0 0" rpy="0 1.57 0" />
+    </joint>
+    <link name="${prefix}intel_camera_depth_optical_frame" />
     <joint name="${prefix}gripper_left_joint" type="prismatic">
       <parent link="${prefix}link5" />

File: src/mobman_description/urdf/turtlebot3_waffle_pi.urdf.xacro (robot description, xacro)
@@ -263,37 +263,5 @@
       <origin xyz="0.003 0.011 0.009" rpy="0 0 0" />
     </joint>
-    <link name="${prefix}camera_rgb_frame">
-      <sensor name="depth_camera" type="rgbd_camera">
-        <always_on>true</always_on>
-        <visualize>true</visualize>
-        <update_rate>5.0</update_rate>
-        <topic>depth_camera</topic>
-        <gz_frame_id>camera_link</gz_frame_id>
-        <camera>
-          <horizontal_fov>1.047198</horizontal_fov>
-          <image>
-            <width>640</width>
-            <height>480</height>
-          </image>
-          <clip>
-            <near>0.05</near>
-            <far>3</far>
-          </clip>
-        </camera>
-        <baseline>0.2</baseline>
-        <pointCloudCutoff>0.5</pointCloudCutoff>
-        <pointCloudCutoffMax>3.0</pointCloudCutoffMax>
-        <distortionK1>0</distortionK1>
-        <distortionK2>0</distortionK2>
-        <distortionK3>0</distortionK3>
-        <distortionT1>0</distortionT1>
-        <distortionT2>0</distortionT2>
-        <CxPrime>0</CxPrime>
-        <Cx>0</Cx>
-        <Cy>0</Cy>
-        <focalLength>0</focalLength>
-        <hackBaseline>0</hackBaseline>
-      </sensor>
-    </link>
+    <link name="${prefix}camera_rgb_frame" />
     <joint name="${prefix}camera_rgb_optical_joint" type="fixed">
       <parent link="${prefix}camera_rgb_frame" />
