Commit message: Modified Rviz for using both Nav2 and Moveit2

File: src/mobman_moveit_config/config/mobman.ros2_control.xacro (robot description, xacro)
@@ -6,6 +6,20 @@
             <hardware>
                 <!-- By default, set up controllers for simulation. This won't work on real hardware -->
-                <plugin>gz_ros2_control/GazeboSimSystem</plugin>
+                <plugin>mock_components/GenericSystem</plugin>
             </hardware>
+            <joint name="gripper_left_joint">
+                <command_interface name="position"/>
+                <state_interface name="position">
+                  <param name="initial_value">${initial_positions['gripper_left_joint']}</param>
+                </state_interface>
+                <state_interface name="velocity"/>
+            </joint>
+            <joint name="gripper_right_joint">
+                <command_interface name="position"/>
+                <state_interface name="position">
+                  <param name="initial_value">${initial_positions['gripper_right_joint']}</param>
+                </state_interface>
+                <state_interface name="velocity"/>
+            </joint>
             <joint name="joint1">
                 <command_interface name="position"/>
@@ -36,11 +50,4 @@
                 <state_interface name="velocity"/>
             </joint>
-            <joint name="gripper_left_joint">
-                <command_interface name="position"/>
-                <state_interface name="position">
-                  <param name="initial_value">${initial_positions['gripper_left_joint']}</param>
-                </state_interface>
-                <state_interface name="velocity"/>
-            </joint>
         </ros2_control>
     </xacro:macro>

File: src/mobman_moveit_config/config/mobman.urdf.xacro (robot description, xacro)
@@ -2,9 +2,8 @@
 <robot xmlns:xacro="http://www.ros.org/wiki/xacro" name="mobman">
     <xacro:arg name="initial_positions_file" default="initial_positions.yaml" />
-    <xacro:arg name="controller_params_file" default="" />
     <!-- Import mobman urdf file -->
     <xacro:include filename="$(find mobman_description)/urdf/mobman.urdf.xacro" />
     <!-- Import control_xacro -->
     <xacro:include filename="mobman.ros2_control.xacro" />
-    <xacro:mobman_ros2_control name="GazeboSimSystem" initial_positions_file="$(arg initial_positions_file)"/>
+    <xacro:mobman_ros2_control name="FakeSystem" initial_positions_file="$(arg initial_positions_file)"/>
 </robot>
